Commit message: Add limit tags to prismatic joints

File: MFR_benchmark/assets/screwdriver/screwdriver_6d_isaaclab.urdf (robot description, URDF)
Before this commit: robot screwdriver_on_the_table, 9 links, 8 joints
Joints:
- joint table_screwdriver_joint_1: limit (none) -> lower=-0.5 upper=0.5 effort=100 velocity=1.0
- joint table_screwdriver_joint_2: limit (none) -> lower=-0.5 upper=0.5 effort=100 velocity=1.0
- joint table_screwdriver_joint_3: limit (none) -> lower=-0.5 upper=0.5 effort=100 velocity=1.0
