Commit message: Added a visual marker for rotation on the model ( no collision volume)

File: MFR_benchmark/assets/screwdriver/screwdriver_isaaclab.urdf (robot description, URDF)
Before this commit: robot screwdriver_on_the_table, 6 links, 5 joints
Links:
- added link marker, mass 0.00001; visual cylinder length=0.1 radius=0.005
Joints:
- added joint screwdriver_body_marker_joint: type fixed, parent screwdriver_body, child marker, origin xyz=0 0 0 rpy=0 0 0, axis 0 0 1
- joint screwdriver_body_cap_joint: type revolute -> continuous
- joint table_screwdriver_joint_3: type revolute -> continuous
